File: ImmunoprecipitationDevice_RevC.kicad_pcb (KiCad board)
At the start: 4 copper layers, 246 x 127 mm, 356 parts

Commit message: Add Revision D - includes scaling changes for multilayer alignment
Other:
- board size 246 x 127 mm -> 100 x 100 mm
- board text added: "C2"
- board text added: "C3"
- board text added: "C4"
- board text added: "F2"
- board text added: "F3"
- board text added: "F4"
